File: DeflectionCoilDrivers/opa548_revised/opa548_revised.kicad_pcb (KiCad board)
At the start: 2 copper layers, 86.5 x 65.6 mm, 49 parts, among them J1 Conn_Coaxial_Small, J2 Conn_01x06_Socket, J5 Conn_Coaxial_Small, U1 OPA548T, U2 OPA548T, U3 OPA1612AID, U4 INA253, U5 L78L05_SO8

Commit message: Fixed footprint references
Parts:
- removed U2: OPA548T, my_local_lib:KVT7
- added C11: 1200pf, Capacitor_SMD:C_0603_1608Metric_Pad1.08x0.95mm_HandSolder, F.Cu at (121.3, 57.1)
- added C3: 1200pf, Capacitor_SMD:C_0603_1608Metric_Pad1.08x0.95mm_HandSolder, F.Cu at (122.1, 66.2)
- added JP1: SolderJumper_2_Open, Jumper:SolderJumper-2_P1.3mm_Open_RoundedPad1.0x1.5mm, F.Cu at (126.5, 65.5)
- added JP4: SolderJumper_2_Open, Jumper:SolderJumper-2_P1.3mm_Open_RoundedPad1.0x1.5mm, F.Cu at (117.8, 63.9)
- added JP5: SolderJumper_2_Open, Jumper:SolderJumper-2_P1.3mm_Open_RoundedPad1.0x1.5mm, F.Cu at (126.4, 56.5)
- added JP6: SolderJumper_2_Open, Jumper:SolderJumper-2_P1.3mm_Open_RoundedPad1.0x1.5mm, F.Cu at (117.0, 55.0)
- added R12: optional, Resistor_SMD:R_0603_1608Metric_Pad0.98x0.95mm_HandSolder, F.Cu at (122.1, 63.9)
- added R13: optional, Resistor_SMD:R_0603_1608Metric_Pad0.98x0.95mm_HandSolder, F.Cu at (121.3, 55.1)
- added RV4: R_Potentiometer_US, Potentiometer_SMD:Potentiometer_Bourns_3269P_Horizontal, F.Cu at (133.5, 65.4)
- added RV5: R_Potentiometer_US, Potentiometer_SMD:Potentiometer_Bourns_3269P_Horizontal, F.Cu at (133.4, 56.6)
- added TP2: TestPoint, Connector_PinSocket_2.54mm:PinSocket_1x01_P2.54mm_Vertical, F.Cu at (98.5, 70.0)
- added U6: ~, Library:opa548, F.Cu at (128.8, 39.1)
- TP1: footprint Connector_PinHeader_1.00mm:PinHeader_1x01_P1.00mm_Vertical -> Connector_PinSocket_2.54mm:PinSocket_1x01_P2.54mm_Vertical
- U1: value OPA548T -> ~; footprint my_local_lib:KVT7 -> Library:opa548
- U3: footprint my_local_lib:D8 -> Library:opa1612
- moved J5 10.8 mm to (126.3, 78.0)
- moved U1 9.98 mm to (93.8, 39.4)
- moved JP2 3.31 mm to (123.3, 49.5)
- moved R15 3.31 mm to (127.9, 50.5)
- moved R14 3.31 mm to (127.9, 48.0)
Routing:
- net Net-(JP3-B): track 38.1 -> 85.2 mm, vias 2 -> 4
- net Net-(JP6-A): track 17.6 -> 46.1 mm, vias 0 -> 2
- net GND: track 27.8 -> 45.1 mm, vias 42 -> 44
- net Net-(JP5-B): track 0.00 -> 16.7 mm, vias 0 -> 2
- net Net-(JP1-B): track 0.00 -> 15.9 mm, vias 0 -> 2
- net +24V: track 188.1 -> 172.7 mm
- net Net-(J5-Ext): track 63.1 -> 73.8 mm
- net Net-(J5-In): track 49.4 -> 56.8 mm
- net Net-(JP24-A): track 6.10 -> 11.5 mm
- net Net-(JP4-B): track 0.00 -> 5.30 mm
- net Net-(JP6-B): track 0.00 -> 5.23 mm
- net -24V: track 208.1 -> 204.9 mm
- net Net-(C3-Pad2): track 0.00 -> 2.32 mm
- net Net-(C11-Pad2): track 0.00 -> 2.02 mm
- net Ilim: track 56.6 -> 55.7 mm
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