File: DeflectionCoilDrivers/opa548_revised/opa548_revised.kicad_sch (KiCad schematic)
At the start: 60 parts, among them J1 Conn_Coaxial_Small, J2 Conn_01x06_Socket, J5 Conn_Coaxial_Small, U1 OPA548T, U2 OPA548T, U3 OPA1612AID, U4 INA253, U5 L78L05_SO8

Commit message: Fixed footprint references
Parts:
- removed U1, U2: OPA548T, my_local_lib:KVT7, symbol 2024-04-29_03-14-05:OPA548T
- added U1, U6: ~, Library:opa548, symbol New_Library:OPA548
- U3: footprint my_local_lib:D8 -> Library:opa1612
Connections:
- net +24V: now also U1.5, U6.5
- net -24V: now also U1.4, U6.4
- net GND: now also U6.1
- net Ilim: now also U1.3, U6.3
- net at JP6.1 (A), R7.2, R9.1: now also U1.1
- net at R5.1, R6.2: now also U1.2
- net at R10.2, R6.1, R8.1: now also U1.6
- net at JP23.2 (B): now also U1.7
- net at J5.2 (Ext), R11.1: now also U6.6
- net at R10.1, R11.2: now also U6.2
- net at JP22.2 (B): now also U6.7
Other:
- moved on the sheet: JP22, JP23
