File: SubstitutionBoard/inductor_board/inductor_board.kicad_sch (KiCad schematic)
At the start: 186 parts, among them J1 Conn_Coaxial_Power, J2 Barrel_Jack_Switch, J3 Conn_01x18, J4 Conn_01x06_Socket, K1 FINDER-32.21-x000, K10 FINDER-32.21-x000, K11 FINDER-32.21-x000, K12 FINDER-32.21-x000, K13 FINDER-32.21-x000, K14 FINDER-32.21-x000, K15 FINDER-32.21-x000, K16 FINDER-32.21-x000, K2 FINDER-32.21-x000, K3 FINDER-32.21-x000, K4 FINDER-32.21-x000, K5 FINDER-32.21-x000, K6 FINDER-32.21-x000, K7 FINDER-32.21-x000, K8 FINDER-32.21-x000, K9 FINDER-32.21-x000, SW1 SW_DIP_x08, SW2 SW_DIP_x08, U1 TLP175A, U10 LM317_SOT-223, U11 TLP175A, U12 LM317_SOT-223, U13 TLP175A, U14 LM317_SOT-223, U15 TLP175A, U16 LM317_SOT-223, U17 TLP175A, U18 LM317_SOT-223, U19 TLP175A, U2 LM317_SOT-223, U20 LM317_SOT-223, U21 TLP175A, U22 LM317_SOT-223, U23 TLP175A, U24 LM317_SOT-223, U25 TLP175A, U26 LM317_SOT-223, U27 TLP175A, U28 LM317_SOT-223, U29 TLP175A, U3 TLP175A, U30 LM317_SOT-223, U31 TLP175A, U32 LM317_SOT-223, U33 L7805, U4 LM317_SOT-223, U5 TLP175A, U6 LM317_SOT-223, U7 TLP175A, U8 LM317_SOT-223, U9 TLP175A

Commit message: Updates
Updated to include both NC and NO solder jumpers for more options. Also added power LED. Also moved power connector closer to edge.
Parts:
- added D17: LED, LED_SMD:LED_0603_1608Metric_Pad1.05x0.95mm_HandSolder, symbol Device:LED
- added JP19, JP20, JP21, JP22, JP23, JP24, JP25, JP26, JP27, JP28, JP29, JP30, JP31, JP32, JP33, JP34, JP35, JP36, JP37, JP38, JP39, JP40, JP41, JP42, JP43, JP44, JP45, JP46, JP47, JP48, JP49, JP50: SolderJumper_2_Open, Jumper:SolderJumper-2_P1.3mm_Open_RoundedPad1.0x1.5mm, symbol Jumper:SolderJumper_2_Open
- added R65: 750, Resistor_SMD:R_0603_1608Metric_Pad0.98x0.95mm_HandSolder, symbol Device:R_Small
Connections:
- net +5V: now also R65.1
- net GND: now also D17.1 (K)
- net Input: now also JP19.1 (A), JP20.1 (A); no longer K1.12
- net at JP5.2 (B), JP6.1 (A), K5.11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: now also JP29.1 (A), JP30.1 (A); no longer K6.12
- net at JP6.2 (B), JP7.1 (A), K6.11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: now also JP31.1 (A), JP32.1 (A); no longer K7.12
- net at JP10.2 (B), JP11.1 (A), K10.11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: now also JP39.1 (A), JP40.1 (A); no longer K11.12
- net at JP11.2 (B), JP12.1 (A), K11.11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: now also JP41.1 (A), JP42.1 (A); no longer K12.12
- net at JP15.2 (B), JP16.1 (A), K15.11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: now also JP49.1 (A), JP50.1 (A); no longer K16.12
- net at K16.14: now also JP50.2 (B)
- net at JP14.2 (B), JP15.1 (A), K14.11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: now also JP47.1 (A), JP48.1 (A); no longer K15.12
- net at JP8.2 (B), JP9.1 (A), K8.11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: now also JP35.1 (A), JP36.1 (A); no longer K9.12
- net at JP10.1 (A), JP9.2 (B), K9.11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: now also JP37.1 (A), JP38.1 (A); no longer K10.12
- net at JP13.2 (B), JP14.1 (A), K13.11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: now also JP45.1 (A), JP46.1 (A); no longer K14.12
- net at K14.14: now also JP46.2 (B)
- net at JP7.2 (B), JP8.1 (A), K7.11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: now also JP33.1 (A), JP34.1 (A); no longer K8.12
- net at JP12.2 (B), JP13.1 (A), K12.11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: now also JP43.1 (A), JP44.1 (A); no longer K13.12
- net at JP3.2 (B), JP4.1 (A), K3.11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: now also JP25.1 (A), JP26.1 (A); no longer K4.12
- net at JP2.2 (B), JP3.1 (A), K2.11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: now also JP23.1 (A), JP24.1 (A); no longer K3.12
- net at K3.14: now also JP24.2 (B)
- net at K8.14: now also JP34.2 (B)
- net at JP1.2 (B), JP2.1 (A), K1.11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: now also JP21.1 (A), JP22.1 (A); no longer K2.12
- net at K13.14: now also JP44.2 (B)
- net at K7.14: now also JP32.2 (B)
- net at JP4.2 (B), JP5.1 (A), K4.11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: now also JP27.1 (A), JP28.1 (A); no longer K5.12
- net at K2.14: now also JP22.2 (B)
- net at K12.14: now also JP42.2 (B)
- net at K15.14: now also JP48.2 (B)
- net at K10.14: now also JP38.2 (B)
- net at K9.14: now also JP36.2 (B)
- net at K5.14: now also JP28.2 (B)
- net at K6.14: now also JP30.2 (B)
- net at K1.14: now also JP20.2 (B)
- net at K11.14: now also JP40.2 (B)
- net at K4.14: now also JP26.2 (B)
- new net: JP49.2 (B), K16.12
- new net: JP45.2 (B), K14.12
- new net: D17.2 (A), R65.2
- new net: JP23.2 (B), K3.12
- new net: JP41.2 (B), K12.12
- new net: JP33.2 (B), K8.12
- new net: JP43.2 (B), K13.12
- new net: JP27.2 (B), K5.12
- new net: JP35.2 (B), K9.12
- new net: JP25.2 (B), K4.12
- new net: JP31.2 (B), K7.12
- new net: JP39.2 (B), K11.12
- new net: JP21.2 (B), K2.12
- new net: JP37.2 (B), K10.12
- new net: JP47.2 (B), K15.12
- new net: JP19.2 (B), K1.12
- new net: JP29.2 (B), K6.12
